Commit message: dividing into seperate nodes + adding collision avoid

File: turtlebot3_description/urdf/turtlebot3_burger.urdf.xacro (robot description, xacro)
@@ -96,6 +96,6 @@
       <origin xyz="0 0.001 0" rpy="0 0 0"/>
       <geometry>
-        <sphere radius="0.004"/>
-        <!-- <box size="0.030 0.009 0.020"/> -->
+        <!-- <sphere radius="0.004"/> -->
+        <box size="0.030 0.009 0.020"/>
       </geometry>
     </collision>

File: turtlebot3_description/urdf/turtlebot3_waffle.gazebo.xacro (robot description, xacro)
@@ -54,5 +54,5 @@
   <gazebo>
     <plugin name="turtlebot3_waffle_controller" filename="libgazebo_ros_diff_drive.so">
-      <commandTopic>cmd_vel</commandTopic>
+      <commandTopic>cmd_vel2</commandTopic>
       <odometryTopic>odom</odometryTopic>
       <odometryFrame>odom</odometryFrame>
