Commit message: .

File: rb1_description/urdf/rb1_description.urdf.xacro (robot description, xacro)
@@ -178,5 +178,5 @@
         <parent link="base_link"/>
         <child link="base_scan"/>
-        <origin xyz="-0.032 0 1" rpy="0 0 0"/>
+        <origin xyz="0 0 1" rpy="0 0 0"/>
     </joint>
     <link name="base_scan">
